Commit message: Finish stage 2 of Rotors-DJI integration.

File: urdf/rotors/dji_m100.urdf.xacro (robot description, xacro)
@@ -4,10 +4,3 @@
   <!-- Instantiate dji_m100 "mechanics" -->
   <xacro:include filename="$(find dji_m100_description)/urdf/rotors/dji_m100_base.xacro" />
-  <!-- Instantiate a controller. -->
-  <xacro:controller_plugin_macro namespace="${namespace}" imu_sub_topic="imu" />
-  <!-- Mount an ADIS16448 IMU. -->
-  <xacro:default_imu namespace="${namespace}" parent_link="${namespace}/base_link" />
-  <xacro:if value="$(arg enable_ground_truth)">
-    <xacro:ground_truth_imu_and_odometry namespace="${namespace}" parent_link="${namespace}/base_link" />
-  </xacro:if>
 </robot>

File: urdf/rotors/dji_m100_base.xacro (robot description, xacro)
@@ -2,5 +2,5 @@
 <robot name="dji_m100" xmlns:xacro="http://ros.org/wiki/xacro">
   <!-- Properties -->
-  <xacro:property name="namespace" value="$(arg namespace)" />
+  <xacro:property name="namespace" value="$(arg robot_namespace)" />
   <xacro:property name="rotor_velocity_slowdown_sim" value="10" />
   <xacro:property name="use_mesh_file" value="true" />
@@ -128,11 +128,24 @@
   </xacro:vertical_rotor>
   <gazebo>
-    <plugin name="ground_truth_plugin" filename="libgazebo_ros_p3d.so">
+    <!-- Possibly noisy odometry sensor attached to the robot-->
+    <plugin name="odometry_sensor_plugin" filename="libgazebo_ros_p3d.so">
+      <robotNamespace>/${namespace}</robotNamespace>
       <bodyName>${namespace}/base_link</bodyName>
       <topicName>odometry</topicName>
       <frameName>/world</frameName>
-      <gaussianNoise>0</gaussianNoise>
-      <updateRate>10</updateRate>
+      <gaussianNoise>0.01</gaussianNoise>
+      <updateRate>50</updateRate>
+    </plugin>
+    <!-- Possibly noisy IMU sensor attached to the robot-->
+    <plugin name="imu_sensor_plugin" filename="libgazebo_ros_imu.so">
+      <alwaysOn>true</alwaysOn>
+      <bodyName>${namespace}/base_link</bodyName>
+      <topicName>imu</topicName>
+      <serviceName>imu_service</serviceName>
+      <gaussianNoise>0.01</gaussianNoise>
+      <updateRate>50</updateRate>
     </plugin>
   </gazebo>
+  <!-- Instantiate a controller. -->
+  <xacro:controller_plugin_macro namespace="${namespace}" imu_sub_topic="imu" />
 </robot>
