Commit message: Parameterize collision and HITL modes.

File: urdf/dji_m100.urdf.xacro (robot description, xacro)
@@ -1,4 +1,6 @@
 <?xml version="1.0"?>
 <robot name="dji_m100" xmlns:xacro="http://www.ros.org/wiki/xacro">
+    <xacro:arg name="robot_namespace" default=""/>
+    <xacro:property name="namespace" value="$(arg robot_namespace)"/>
     <xacro:include filename="$(find dji_m100_description)/urdf/dji_m100_base.xacro" />
     <xacro:include filename="$(find dji_m100_description)/urdf/gimbal.urdf.xacro" />

File: urdf/dji_m100_base.xacro (robot description, xacro)
@@ -1,5 +1,6 @@
 <?xml version="1.0"?>
 <robot xmlns:xacro="http://www.ros.org/wiki/xacro">
-  <xacro:property name="pi" value="3.1415926535897931" />
+  <xacro:arg name="hitl_model" default="true"/>
+  <xacro:arg name="collision_enabled" default="false"/>
   <xacro:property name="M_PI" value="3.1415926535897931" />
  <!-- Base quadrotor link -->
@@ -11,8 +12,14 @@
         <inertia ixx="0.11152" ixy="0.0" ixz="0.0" iyy="0.11152" iyz="0.0" izz="0.218" />
       </inertial>
-      <visual>
+      <visual name="body">
         <origin xyz="0 0 0" rpy="0 0 0" />
         <geometry>
           <mesh filename="package://dji_m100_description/meshes/dji_m100/dji_m100.dae"/>
+        </geometry>
+      </visual>
+      <visual name="base_link::collision_sphere">
+        <pose frame=''>0 0 0 0 0 0</pose>
+        <geometry>
+          <sphere radius="0.75"/>
         </geometry>
       </visual>
@@ -25,10 +32,36 @@
       <gravity>1</gravity>
     </link>
-    <!-- DJI Gazebo Controller Plugin -->
-    <gazebo>
-      <plugin name='dji_ros_gazebo_controller' filename='libdji_ros_gazebo_control.so'>
-        <allow_contact_sensing>false</allow_contact_sensing> <!-- If you want to enable contact sensing make it true -->
-      </plugin>
-    </gazebo>
+    <!-- HITL model config -->
+    <xacro:if value="$(arg hitl_model)">
+      <!-- Add illustrative transparent sphere around the drone -->
+      <gazebo reference="base_link">
+        <visual name="base_link::collision_sphere">
+          <material>
+            <ambient>1 0 0 0.3</ambient>
+            <diffuse>1 0 0 0.3</diffuse>
+            <specular>1 0 0 0.3</specular>
+            <emissive>0 0 0 0.3</emissive>
+          </material>
+        </visual>
+      </gazebo>
+      <!-- DJI Gazebo Controller Plugin -->
+      <gazebo>
+        <plugin name='dji_ros_gazebo_controller' filename='libdji_ros_gazebo_control.so'>
+          <allow_contact_sensing>$(arg collision_enabled)</allow_contact_sensing> <!-- If you want to enable contact sensing make it true -->
+        </plugin>
+      </gazebo>
+    </xacro:if>
+    <xacro:unless value="$(arg hitl_model)">
+      <gazebo reference="base_link">
+      <visual name="base_link::collision_sphere">
+          <material>
+            <ambient>0 0 1 0.3</ambient>
+            <diffuse>0 0 1 0.3</diffuse>
+            <specular>0 0 1 0.3</specular>
+            <emissive>0 0 0 0.3</emissive>
+          </material>
+        </visual>
+      </gazebo>
+    </xacro:unless>
     <!-- Contact sensor -->
     <gazebo reference="base_link">

Commit message: Reduce repetitions, add more parameterization to get closer finishing integration.

File: urdf/dji_m100.urdf.xacro (robot description, xacro)
@@ -5,5 +5,5 @@
     <xacro:include filename="$(find dji_m100_description)/urdf/dji_m100_base.xacro" />
     <xacro:include filename="$(find dji_m100_description)/urdf/gimbal.urdf.xacro" />
-    <xacro:dji_m100_base_macro />
+    <xacro:dji_m100_body />
     <xacro:dji_m100_gimbal />
 </robot>

File: urdf/dji_m100_base.xacro (robot description, xacro)
@@ -1,35 +1,138 @@
 <?xml version="1.0"?>
-<robot xmlns:xacro="http://www.ros.org/wiki/xacro">
+<robot name="dji_m100" xmlns:xacro="http://ros.org/wiki/xacro">
+  <!-- Arguments -->
   <xacro:arg name="hitl_model" default="true"/>
   <xacro:arg name="collision_enabled" default="false"/>
-  <xacro:property name="M_PI" value="3.1415926535897931" />
- <!-- Base quadrotor link -->
-  <xacro:macro name="dji_m100_base_macro">
-    <link name="base_link">
-      <inertial>
-        <mass value="1024" />
-        <origin xyz="0 0 0" />
-        <inertia ixx="170.667" ixy="0.0" ixz="0.0" iyy="170.667" iyz="0.0" izz="170.667" />
-      </inertial>
-      <visual name="body">
-        <origin xyz="0 0 0" rpy="0 0 0" />
-        <geometry>
-          <mesh filename="package://dji_m100_description/meshes/dji_m100/dji_m100.dae"/>
-        </geometry>
-      </visual>
-      <visual name="base_link::collision_sphere">
-        <pose frame=''>0 0 0 0 0 0</pose>
-        <geometry>
-          <sphere radius="0.75"/>
-        </geometry>
-      </visual>
-      <collision>
-        <origin xyz="0 0 0" rpy="0 0 0" />
-        <geometry>
-          <mesh filename="package://dji_m100_description/meshes/dji_m100/dji_m100.stl"/>
-        </geometry>
-      </collision>
-      <gravity>1</gravity>
-    </link>
+  <xacro:arg name="rotors_controlled" default="false"/>
+  <!-- Properties -->
+  <xacro:property name="namespace" value="$(arg robot_namespace)" />
+  <xacro:property name="rotor_velocity_slowdown_sim" value="10" />
+  <xacro:property name="use_mesh_file" value="true" />
+  <xacro:property name="mesh_file" value="package://dji_m100_description/meshes/dji_m100/dji_m100_flipped_rotorless.dae" />
+  <xacro:property name="mass" value="2.355" /> <!-- [kg] -->
+  <xacro:property name="body_width" value="0.3" /> <!-- [m] / This value is not important since we've already provided the mesh. -->
+  <xacro:property name="body_height" value="0.16" /> <!-- [m] / This value is not important since we've already provided the mesh. -->
+  <xacro:property name="mass_rotor" value="0.08" /> <!-- [kg] -->
+  <xacro:property name="arm_length" value="0.17" /> <!-- [m] -->
+  <xacro:property name="rotor_offset_top" value="0.1" /> <!-- [m] -->
+  <xacro:property name="radius_rotor" value="0.195" /> <!-- [m] -->
+  <xacro:property name="motor_constant" value="1.84858e-05" /> <!-- [kg.m/s^2] -->
+  <xacro:property name="moment_constant" value="0.016" /> <!-- [m] -->
+  <xacro:property name="time_constant_up" value="0.0125" /> <!-- [s] -->
+  <xacro:property name="time_constant_down" value="0.025" /> <!-- [s] -->
+  <xacro:property name="max_rot_velocity" value="838" /> <!-- [rad/s] -->
+  <xacro:property name="sin30" value="0.5" />
+  <xacro:property name="cos30" value="0.866025403784" />
+  <xacro:property name="sqrt2" value="1.4142135623730951" />
+  <xacro:property name="rotor_drag_coefficient" value="8.06428e-05" />
+  <xacro:property name="rolling_moment_coefficient" value="0.000001" />
+  <!-- Property Blocks -->
+  <xacro:property name="body_inertia">
+    <inertia ixx="0.1547563" ixy="0.0" ixz="0.0" iyy="0.1658929" iyz="0.0" izz="0.2077" /> <!-- [kg.m^2] [kg.m^2] [kg.m^2] [kg.m^2] [kg.m^2] [kg.m^2] -->
+  </xacro:property>
+  <!-- inertia of a single rotor, assuming it is a cuboid. Height=3mm, width=15mm -->
+  <xacro:property name="rotor_inertia">
+    <xacro:box_inertia x="${radius_rotor}" y="0.015" z="0.003" mass="${mass_rotor*rotor_velocity_slowdown_sim}" />
+  </xacro:property>
+  <!-- Included URDF Files -->
+  <xacro:include filename="$(find rotors_description)/urdf/component_snippets.xacro" />
+  <xacro:include filename="$(find rotors_description)/urdf/multirotor_base.xacro" />
+  <xacro:macro name="dji_m100_body">
+    <!-- Instantiate multirotor_base_macro once -->
+    <xacro:multirotor_base_macro
+      robot_namespace="${namespace}"
+      mass="${mass}"
+      body_width="${body_width}"
+      body_height="${body_height}"
+      use_mesh_file="${use_mesh_file}"
+      mesh_file="${mesh_file}"
+      >
+      <xacro:insert_block name="body_inertia" />
+    </xacro:multirotor_base_macro>
+    <!-- Instantiate rotors -->
+    <xacro:vertical_rotor
+      robot_namespace="${namespace}"
+      suffix="front_right"
+      direction="ccw"
+      motor_constant="${motor_constant}"
+      moment_constant="${moment_constant}"
+      parent="${namespace}/base_link"
+      mass_rotor="${mass_rotor}"
+      radius_rotor="${radius_rotor}"
+      time_constant_up="${time_constant_up}"
+      time_constant_down="${time_constant_down}"
+      max_rot_velocity="${max_rot_velocity}"
+      motor_number="0"
+      rotor_drag_coefficient="${rotor_drag_coefficient}"
+      rolling_moment_coefficient="${rolling_moment_coefficient}"
+      color="Black"
+      use_own_mesh="false"
+      mesh="">
+      <origin xyz="${sqrt2 * arm_length} -${sqrt2 * arm_length} ${rotor_offset_top}" rpy="0 0 0" />
+      <xacro:insert_block name="rotor_inertia" />
+    </xacro:vertical_rotor>
+    <xacro:vertical_rotor
+      robot_namespace="${namespace}"
+      suffix="back_left"
+      direction="ccw"
+      motor_constant="${motor_constant}"
+      moment_constant="${moment_constant}"
+      parent="${namespace}/base_link"
+      mass_rotor="${mass_rotor}"
+      radius_rotor="${radius_rotor}"
+      time_constant_up="${time_constant_up}"
+      time_constant_down="${time_constant_down}"
+      max_rot_velocity="${max_rot_velocity}"
+      motor_number="1"
+      rotor_drag_coefficient="${rotor_drag_coefficient}"
+      rolling_moment_coefficient="${rolling_moment_coefficient}"
+      color="Black"
+      use_own_mesh="false"
+      mesh="">
+      <origin xyz="-${sqrt2 * arm_length} ${sqrt2 * arm_length} ${rotor_offset_top}" rpy="0 0 0" />
+      <xacro:insert_block name="rotor_inertia" />
+    </xacro:vertical_rotor>
+    <xacro:vertical_rotor
+      robot_namespace="${namespace}"
+      suffix="front_left"
+      direction="cw"
+      motor_constant="${motor_constant}"
+      moment_constant="${moment_constant}"
+      parent="${namespace}/base_link"
+      mass_rotor="${mass_rotor}"
+      radius_rotor="${radius_rotor}"
+      time_constant_up="${time_constant_up}"
+      time_constant_down="${time_constant_down}"
+      max_rot_velocity="${max_rot_velocity}"
+      motor_number="2"
+      rotor_drag_coefficient="${rotor_drag_coefficient}"
+      rolling_moment_coefficient="${rolling_moment_coefficient}"
+      color="Black"
+      use_own_mesh="false"
+      mesh="">
+      <origin xyz="${sqrt2 * arm_length} ${sqrt2 * arm_length} ${rotor_offset_top}" rpy="0 0 0" />
+      <xacro:insert_block name="rotor_inertia" />
+    </xacro:vertical_rotor>
+    <xacro:vertical_rotor
+      robot_namespace="${namespace}"
+      suffix="back_right"
+      direction="cw"
+      motor_constant="${motor_constant}"
+      moment_constant="${moment_constant}"
+      parent="${namespace}/base_link"
+      mass_rotor="${mass_rotor}"
+      radius_rotor="${radius_rotor}"
+      time_constant_up="${time_constant_up}"
+      time_constant_down="${time_constant_down}"
+      max_rot_velocity="${max_rot_velocity}"
+      motor_number="3"
+      rotor_drag_coefficient="${rotor_drag_coefficient}"
+      rolling_moment_coefficient="${rolling_moment_coefficient}"
+      color="Black"
+      use_own_mesh="false"
+      mesh="">
+      <origin xyz="-${sqrt2 * arm_length} -${sqrt2 * arm_length} ${rotor_offset_top}" rpy="0 0 0" />
+      <xacro:insert_block name="rotor_inertia" />
+    </xacro:vertical_rotor>
     <!-- HITL model config -->
     <xacro:if value="$(arg hitl_model)">
@@ -53,4 +156,5 @@
       </gazebo>
     </xacro:if>
+    <!-- SITL model config -->
     <xacro:unless value="$(arg hitl_model)">
       <gazebo reference="base_link">
@@ -64,36 +168,60 @@
         </visual>
       </gazebo>
+      <!-- Instantiate a controller. -->
+      <xacro:if value="$(arg rotors_controlled)">
+        <xacro:controller_plugin_macro namespace="${namespace}" imu_sub_topic="imu" />
+      </xacro:if>
+      <xacro:unless value="$(arg rotors_controlled)">
+        <gazebo>
+          <plugin name="sitl_controller" filename="libgazebo_ros_control.so">
+            <controlPeriod>0.01</controlPeriod>
+            <robotSimType>dji_m100_controller_gazebo_sitl/DJIM100HardwareSim</robotSimType>
+            <allow_contact_sensing>$(arg collision_enabled)</allow_contact_sensing>
+          </plugin>
+        </gazebo>
+      </xacro:unless>
+      <!-- Battery -->
+      <gazebo reference="base_link">
+        <battery name="linear_battery">
+          <voltage>12.592</voltage>
+        </battery>
+      </gazebo>
       <gazebo>
-        <plugin name="sitl_controller" filename="libgazebo_ros_control.so">
-          <controlPeriod>0.01</controlPeriod>
-          <robotSimType>dji_m100_controller_gazebo_sitl/DJIM100HardwareSim</robotSimType>
-          <allow_contact_sensing>$(arg collision_enabled)</allow_contact_sensing>
-        </plugin>
-      </gazebo>
-      <!-- Battery -->
-    <gazebo reference="base_link">
-      <battery name="linear_battery">
-        <voltage>12.592</voltage>
-      </battery>
-    </gazebo>
-    <gazebo>
-      <!-- Battery voltage tracker -->
-      <plugin name="battery" filename="libLinearBatteryPlugin.so">
-        <link_name>base_link</link_name>
-        <battery_name>linear_battery</battery_name>
-        <open_circuit_voltage_constant_coef>12.694</open_circuit_voltage_constant_coef>
-        <open_circuit_voltage_linear_coef>-6.7424</open_circuit_voltage_linear_coef>
-        <initial_charge>1.1665</initial_charge>
-        <capacity>1.2009</capacity>
-        <resistance>0.061523</resistance>
-        <smooth_current_tau>5.9499</smooth_current_tau>
-      </plugin>
-      <!-- Battery voltage consumer -->
-      <plugin name="motherboard" filename="libLinearBatteryConsumerPlugin.so">
-        <link_name>base_link</link_name>
-        <battery_name>linear_battery</battery_name>
-        <power_load>606.6</power_load>
-      </plugin>
-    </gazebo>
+        <!-- Battery voltage tracker -->
+        <plugin name="battery" filename="libLinearBatteryPlugin.so">
+          <link_name>base_link</link_name>
+          <battery_name>linear_battery</battery_name>
+          <open_circuit_voltage_constant_coef>12.694</open_circuit_voltage_constant_coef>
+          <open_circuit_voltage_linear_coef>-6.7424</open_circuit_voltage_linear_coef>
+          <initial_charge>1.1665</initial_charge>
+          <capacity>1.2009</capacity>
+          <resistance>0.061523</resistance>
+          <smooth_current_tau>5.9499</smooth_current_tau>
+        </plugin>
+        <!-- Battery voltage consumer -->
+        <plugin name="motherboard" filename="libLinearBatteryConsumerPlugin.so">
+          <link_name>base_link</link_name>
+          <battery_name>linear_battery</battery_name>
+          <power_load>606.6</power_load>
+        </plugin>
+        <!-- Noisy odometry sensor attached to the robot-->
+        <plugin name="odometry_sensor_plugin" filename="libgazebo_ros_p3d.so">
+          <robotNamespace>/${namespace}</robotNamespace>
+          <bodyName>${namespace}/base_link</bodyName>
+          <topicName>odometry</topicName>
+          <frameName>/world</frameName>
+          <gaussianNoise>0.01</gaussianNoise>
+          <updateRate>50</updateRate>
+        </plugin>
+        <!-- Noisy IMU sensor attached to the robot-->
+        <plugin name="imu_sensor_plugin" filename="libgazebo_ros_imu.so">
+          <alwaysOn>true</alwaysOn>
+          <bodyName>${namespace}/base_link</bodyName>
+          <topicName>imu</topicName>
+          <serviceName>imu_service</serviceName>
+          <gaussianNoise>0.01</gaussianNoise>
+          <updateRate>50</updateRate>
+        </plugin>
+      </gazebo>
     </xacro:unless>
     <!-- Contact sensor -->
@@ -110,12 +238,13 @@
       </sensor>
     </gazebo>
+    <!-- Ground truth odometry -->
     <gazebo>
-      <plugin name="ground_truth_plugin" filename="libgazebo_ros_p3d.so">
+      <plugin name="ground_truth_odometry" filename="libgazebo_ros_p3d.so">
         <robotNamespace>/${namespace}</robotNamespace>
-        <bodyName>base_link</bodyName>
-        <topicName>odometry</topicName>
+        <bodyName>${namespace}/base_link</bodyName>
+        <topicName>ground_truth/odometry</topicName>
         <frameName>/world</frameName>
         <gaussianNoise>0</gaussianNoise>
-        <updateRate>10</updateRate>
+        <updateRate>20</updateRate>
       </plugin>
     </gazebo>

File: urdf/rotors/dji_m100.urdf.xacro (robot description, xacro)
@@ -1,6 +1,6 @@
 <?xml version="1.0"?>
 <robot name="dji_m100" xmlns:xacro="http://ros.org/wiki/xacro">
-  <xacro:include filename="$(find rotors_description)/urdf/component_snippets.xacro" />
   <!-- Instantiate dji_m100 "mechanics" -->
-  <xacro:include filename="$(find dji_m100_description)/urdf/rotors/dji_m100_base.xacro" />
+  <xacro:include filename="$(find dji_m100_description)/urdf/dji_m100_base.xacro" />
+  <xacro:dji_m100_body />
 </robot>

Commit message: Finalize URDF-integration of Rotors misc to DJI stack.

File: urdf/dji_m100.urdf.xacro (robot description, xacro)
@@ -1,9 +1,11 @@
 <?xml version="1.0"?>
-<robot name="dji_m100" xmlns:xacro="http://www.ros.org/wiki/xacro">
-    <xacro:arg name="robot_namespace" default=""/>
-    <xacro:property name="namespace" value="$(arg robot_namespace)"/>
-    <xacro:include filename="$(find dji_m100_description)/urdf/dji_m100_base.xacro" />
-    <xacro:include filename="$(find dji_m100_description)/urdf/gimbal.urdf.xacro" />
-    <xacro:dji_m100_body />
-    <xacro:dji_m100_gimbal />
+<robot name="dji_m100" xmlns:xacro="http://ros.org/wiki/xacro">
+  <xacro:arg name="robot_namespace" default=""/>
+  <xacro:property name="namespace" value="$(arg robot_namespace)" />
+  <xacro:arg name="complex_visualization_supported" default="true"/>
+  <!-- Instantiate dji_m100 "mechanics" -->
+  <xacro:include filename="$(find dji_m100_description)/urdf/dji_m100_base.xacro" />
+  <xacro:include filename="$(find dji_m100_description)/urdf/gimbal.urdf.xacro" />
+  <xacro:dji_m100_body />
+  <xacro:dji_m100_gimbal />
 </robot>

File: urdf/gimbal.urdf.xacro (robot description, xacro)
@@ -2,4 +2,5 @@
 <robot xmlns:xacro="http://www.ros.org/wiki/xacro">
     <xacro:include filename="$(find dji_m100_description)/urdf/gimbal_joints.xacro"/>
+    <xacro:property name="M_PI" value="3.14"/>
     <xacro:macro name="dji_m100_gimbal">
         <revolute_gimbal_joint
