Commit message: Adjust gimbal pose accordingly.

File: urdf/dji_m100_base.xacro (robot description, xacro)
@@ -28,30 +28,4 @@
     <gazebo>
       <plugin name='dji_ros_gazebo_controller' filename='libdji_ros_gazebo_control.so'>
-        <mode>1</mode> <!-- 0 is XYZ, 1 is GPS -->
-        <bodyName>base_link</bodyName>
-        <imuTopic>dji_sdk/imu</imuTopic>
-        <rollpitchProportionalGain>10.0</rollpitchProportionalGain>
-        <rollpitchDifferentialGain>5.0</rollpitchDifferentialGain>
-        <rollpitchLimit>0.5</rollpitchLimit>
-        <yawProportionalGain>2.0</yawProportionalGain>
-        <yawDifferentialGain>1.0</yawDifferentialGain>
-        <yawLimit>1.5</yawLimit>
-        <velocityXYProportionalGain>5.0</velocityXYProportionalGain>
-        <velocityXYDifferentialGain>2.3</velocityXYDifferentialGain>
-        <velocityXYLimit>2</velocityXYLimit>
-        <velocityZProportionalGain>5.0</velocityZProportionalGain>
-        <velocityZDifferentialGain>1.0</velocityZDifferentialGain>
-        <velocityZLimit>-1</velocityZLimit>
-        <positionXYProportionalGain>1.1</positionXYProportionalGain>
-        <positionXYDifferentialGain>0.0</positionXYDifferentialGain>
-        <positionXYIntegralGain>0.0</positionXYIntegralGain>
-        <positionXYLimit>5</positionXYLimit>
-        <positionZProportionalGain>1.0</positionZProportionalGain>
-        <positionZDifferentialGain>0.2</positionZDifferentialGain>
-        <positionZLimit>-1</positionZLimit>
-        <maxForce>30</maxForce>
-        <motionSmallNoise>0.0</motionSmallNoise>
-        <motionDriftNoise>0.0</motionDriftNoise>
-        <motionDriftNoiseTime>0.0</motionDriftNoiseTime>
       </plugin>
     </gazebo>

File: urdf/gimbal.urdf.xacro (robot description, xacro)
@@ -3,5 +3,5 @@
     <xacro:macro name="dji_m100_gimbal">
         <joint name="virtual_gimbal_joint" type="fixed">
-            <origin xyz="0.1 0 -0.04" rpy="0 0 0"/>
+            <origin xyz="-0.1 0 -0.04" rpy="0 0 0"/>
             <parent link="base_link"/>
             <child link="virtual_gimbal_link"/>
@@ -73,9 +73,9 @@
             <inertial>
                 <mass value="0.0001" />
-                <origin xyz="0 0 0" rpy="0 0 0" />
+                <origin xyz="0 0 0" rpy="0 0 ${-M_PI}" />
                 <inertia ixx="0.0001" ixy="0" ixz="0" iyy="0.0001" iyz="0" izz="0.0001" />
             </inertial>
             <visual>
-                <origin xyz="0 0 0" rpy="0 0 0" />
+                <origin xyz="0 0 0" rpy="0 0 ${-M_PI}" />
                 <geometry>
                 <mesh filename="package://dji_m100_description/meshes/dji_m100/gimbal.dae"/>
@@ -83,5 +83,5 @@
             </visual>
             <collision>
-                <origin xyz="0 0 0" rpy="0 0 0" />
+                <origin xyz="0 0 0" rpy="0 0 ${-M_PI}" />
                 <geometry>
                 <mesh filename="package://dji_m100_description/meshes/dji_m100/gimbal.stl"/>
@@ -113,5 +113,5 @@
                 <!-- <pose>0.027 0 -0.027 0 1.57 0</pose> -->
                 <!-- <pose>0.027 0 -0.027 0 1.57 0</pose> -->
-                <pose>0.027 0 -0.027 0 0 0</pose>
+                <pose>0.107 0 -0.127 0 0 0</pose>
                 <horizontal_fov>${94 * M_PI/180.0}</horizontal_fov>
                 <image>

Commit message: Add contact sensor and adjust camera position.

File: urdf/dji_m100_base.xacro (robot description, xacro)
@@ -30,4 +30,17 @@
       </plugin>
     </gazebo>
+    <!-- Contact sensor -->
+    <gazebo reference="base_link">
+      <sensor name="body_contact_sensor" type="contact">
+        <always_on>true</always_on>
+        <contact>
+          <collision>base_link_collision</collision>
+        </contact>
+        <plugin name="dji_m100_bumper" filename="libgazebo_ros_bumper.so">
+          <bumperTopicName>contact</bumperTopicName>
+          <frameName>base_link</frameName>
+        </plugin>
+      </sensor>
+    </gazebo>
   </xacro:macro>
 </robot>

File: urdf/gimbal.urdf.xacro (robot description, xacro)
@@ -113,5 +113,5 @@
                 <!-- <pose>0.027 0 -0.027 0 1.57 0</pose> -->
                 <!-- <pose>0.027 0 -0.027 0 1.57 0</pose> -->
-                <pose>0.107 0 -0.127 0 0 ${M_PI}</pose>
+                <pose>0.107 0 -0.227 0 0 ${M_PI}</pose>
                 <horizontal_fov>${94 * M_PI/180.0}</horizontal_fov>
                 <image>

Commit message: Important: Since forces on gimbal need to be encountered by a reaction force, the body reacts. In order to remove disturbances, an unrealistic mass is given.

File: urdf/dji_m100_base.xacro (robot description, xacro)
@@ -8,7 +8,7 @@
     <link name="base_link">
       <inertial>
-        <mass value="1.477" />
+        <mass value="1024" />
         <origin xyz="0 0 0" />
-        <inertia ixx="0.11152" ixy="0.0" ixz="0.0" iyy="0.11152" iyz="0.0" izz="0.218" />
+        <inertia ixx="170.667" ixy="0.0" ixz="0.0" iyy="170.667" iyz="0.0" izz="170.667" />
       </inertial>
       <visual name="body">
@@ -55,5 +55,5 @@
     <xacro:unless value="$(arg hitl_model)">
       <gazebo reference="base_link">
-      <visual name="base_link::collision_sphere">
+        <visual name="base_link::collision_sphere">
           <material>
             <ambient>0 0 1 0.3</ambient>
@@ -63,4 +63,7 @@
           </material>
         </visual>
+      </gazebo>
+      <gazebo>
+        <plugin name="gazebo_ros_control" filename="libgazebo_ros_control.so"/>
       </gazebo>
     </xacro:unless>

Commit message: Add namespace to visual name for further reference by gazebo tags.

File: urdf/dji_m100_base.xacro (robot description, xacro)
@@ -12,5 +12,5 @@
         <inertia ixx="170.667" ixy="0.0" ixz="0.0" iyy="170.667" iyz="0.0" izz="170.667" />
       </inertial>
-      <visual name="body">
+      <visual name="base_link::body">
         <origin xyz="0 0 0" rpy="0 0 0" />
         <geometry>

Commit message: Control gimbal through one controller.

File: urdf/dji_m100_base.xacro (robot description, xacro)
@@ -12,5 +12,5 @@
         <inertia ixx="170.667" ixy="0.0" ixz="0.0" iyy="170.667" iyz="0.0" izz="170.667" />
       </inertial>
-      <visual name="base_link::body">
+      <visual name="body">
         <origin xyz="0 0 0" rpy="0 0 0" />
         <geometry>
@@ -47,5 +47,5 @@
       <!-- DJI Gazebo Controller Plugin -->
       <gazebo>
-        <plugin name='dji_ros_gazebo_controller' filename='libdji_ros_gazebo_control.so'>
+        <plugin name='dji_ros_gazebo_controller' filename='libdji_ros_gazebo_control_hitl.so'>
           <allow_contact_sensing>$(arg collision_enabled)</allow_contact_sensing> <!-- If you want to enable contact sensing make it true -->
           <initial_height>1.0</initial_height>
@@ -65,5 +65,7 @@
       </gazebo>
       <gazebo>
-        <plugin name="gazebo_ros_control" filename="libgazebo_ros_control.so"/>
+        <plugin name="sitl_controller" filename="libgazebo_ros_control.so">
+          <controlPeriod>0.01</controlPeriod>
+        </plugin>
       </gazebo>
     </xacro:unless>

Commit message: Customize rotors stuff and locally get them whenever possible. Support Gazebo < 7.0 and 8.0> gracefully.

File: urdf/dji_m100_base.xacro (robot description, xacro)
@@ -6,8 +6,5 @@
   <xacro:arg name="rotors_controlled" default="false"/>
   <!-- Properties -->
-  <xacro:property name="namespace" value="$(arg robot_namespace)" />
   <xacro:property name="rotor_velocity_slowdown_sim" value="10" />
-  <xacro:property name="use_mesh_file" value="true" />
-  <xacro:property name="mesh_file" value="package://dji_m100_description/meshes/dji_m100/dji_m100_flipped_rotorless.dae" />
   <xacro:property name="mass" value="2.355" /> <!-- [kg] -->
   <xacro:property name="body_width" value="0.3" /> <!-- [m] / This value is not important since we've already provided the mesh. -->
@@ -36,18 +33,13 @@
   </xacro:property>
   <!-- Included URDF Files -->
-  <xacro:include filename="$(find rotors_description)/urdf/component_snippets.xacro" />
-  <xacro:include filename="$(find rotors_description)/urdf/multirotor_base.xacro" />
+  <xacro:include filename="$(find dji_m100_description)/urdf/rotors/dji_m100_multirotors.xacro"/>
   <xacro:macro name="dji_m100_body">
-    <!-- Instantiate multirotor_base_macro once -->
-    <xacro:multirotor_base_macro
+    <!-- Instantiate DJI M100 multirotor base macro -->
+    <xacro:dji_m100_multirotor_base
       robot_namespace="${namespace}"
       mass="${mass}"
-      body_width="${body_width}"
-      body_height="${body_height}"
-      use_mesh_file="${use_mesh_file}"
-      mesh_file="${mesh_file}"
       >
       <xacro:insert_block name="body_inertia" />
-    </xacro:multirotor_base_macro>
+    </xacro:dji_m100_multirotor_base>
     <!-- Instantiate rotors -->
     <xacro:vertical_rotor
@@ -57,5 +49,5 @@
       motor_constant="${motor_constant}"
       moment_constant="${moment_constant}"
-      parent="${namespace}/base_link"
+      parent="base_link"
       mass_rotor="${mass_rotor}"
       radius_rotor="${radius_rotor}"
@@ -66,7 +58,5 @@
       rotor_drag_coefficient="${rotor_drag_coefficient}"
       rolling_moment_coefficient="${rolling_moment_coefficient}"
-      color="Black"
-      use_own_mesh="false"
-      mesh="">
+      color="Black">
       <origin xyz="${sqrt2 * arm_length} -${sqrt2 * arm_length} ${rotor_offset_top}" rpy="0 0 0" />
       <xacro:insert_block name="rotor_inertia" />
@@ -78,5 +68,5 @@
       motor_constant="${motor_constant}"
       moment_constant="${moment_constant}"
-      parent="${namespace}/base_link"
+      parent="base_link"
       mass_rotor="${mass_rotor}"
       radius_rotor="${radius_rotor}"
@@ -87,7 +77,5 @@
       rotor_drag_coefficient="${rotor_drag_coefficient}"
       rolling_moment_coefficient="${rolling_moment_coefficient}"
-      color="Black"
-      use_own_mesh="false"
-      mesh="">
+      color="Black">
       <origin xyz="-${sqrt2 * arm_length} ${sqrt2 * arm_length} ${rotor_offset_top}" rpy="0 0 0" />
       <xacro:insert_block name="rotor_inertia" />
@@ -99,5 +87,5 @@
       motor_constant="${motor_constant}"
       moment_constant="${moment_constant}"
-      parent="${namespace}/base_link"
+      parent="base_link"
       mass_rotor="${mass_rotor}"
       radius_rotor="${radius_rotor}"
@@ -108,7 +96,5 @@
       rotor_drag_coefficient="${rotor_drag_coefficient}"
       rolling_moment_coefficient="${rolling_moment_coefficient}"
-      color="Black"
-      use_own_mesh="false"
-      mesh="">
+      color="Black">
       <origin xyz="${sqrt2 * arm_length} ${sqrt2 * arm_length} ${rotor_offset_top}" rpy="0 0 0" />
       <xacro:insert_block name="rotor_inertia" />
@@ -120,5 +106,5 @@
       motor_constant="${motor_constant}"
       moment_constant="${moment_constant}"
-      parent="${namespace}/base_link"
+      parent="base_link"
       mass_rotor="${mass_rotor}"
       radius_rotor="${radius_rotor}"
@@ -129,7 +115,5 @@
       rotor_drag_coefficient="${rotor_drag_coefficient}"
       rolling_moment_coefficient="${rolling_moment_coefficient}"
-      color="Black"
-      use_own_mesh="false"
-      mesh="">
+      color="Black">
       <origin xyz="-${sqrt2 * arm_length} -${sqrt2 * arm_length} ${rotor_offset_top}" rpy="0 0 0" />
       <xacro:insert_block name="rotor_inertia" />
@@ -138,14 +122,16 @@
     <xacro:if value="$(arg hitl_model)">
       <!-- Add illustrative transparent sphere around the drone -->
-      <gazebo reference="base_link">
-        <visual name="base_link::collision_sphere">
-          <material>
-            <ambient>1 0 0 0.3</ambient>
-            <diffuse>1 0 0 0.3</diffuse>
-            <specular>1 0 0 0.3</specular>
-            <emissive>0 0 0 0.3</emissive>
-          </material>
-        </visual>
-      </gazebo>
+      <xacro:if value="$(arg complex_visualization_supported)">
+        <gazebo reference="base_link">
+          <visual name="base_link::collision_sphere">
+            <material>
+              <ambient>1 0 0 0.3</ambient>
+              <diffuse>1 0 0 0.3</diffuse>
+              <specular>1 0 0 0.3</specular>
+              <emissive>0 0 0 0.3</emissive>
+            </material>
+          </visual>
+        </gazebo>
+       </xacro:if>
       <!-- DJI Gazebo Controller Plugin -->
       <gazebo>
@@ -158,14 +144,16 @@
     <!-- SITL model config -->
     <xacro:unless value="$(arg hitl_model)">
-      <gazebo reference="base_link">
-        <visual name="base_link::collision_sphere">
-          <material>
-            <ambient>0 0 1 0.3</ambient>
-            <diffuse>0 0 1 0.3</diffuse>
-            <specular>0 0 1 0.3</specular>
-            <emissive>0 0 0 0.3</emissive>
-          </material>
-        </visual>
-      </gazebo>
+      <xacro:if value="$(arg complex_visualization_supported)">
+        <gazebo reference="base_link">
+          <visual name="base_link::collision_sphere">
+            <material>
+              <ambient>0 0 1 0.3</ambient>
+              <diffuse>0 0 1 0.3</diffuse>
+              <specular>0 0 1 0.3</specular>
+              <emissive>0 0 0 0.3</emissive>
+            </material>
+          </visual>
+        </gazebo>
+      </xacro:if>
       <!-- Instantiate a controller. -->
       <xacro:if value="$(arg rotors_controlled)">
@@ -208,5 +196,5 @@
         <plugin name="odometry_sensor_plugin" filename="libgazebo_ros_p3d.so">
           <robotNamespace>/${namespace}</robotNamespace>
-          <bodyName>${namespace}/base_link</bodyName>
+          <bodyName>base_link</bodyName>
           <topicName>odometry</topicName>
           <frameName>/world</frameName>
@@ -217,5 +205,5 @@
         <plugin name="imu_sensor_plugin" filename="libgazebo_ros_imu.so">
           <alwaysOn>true</alwaysOn>
-          <bodyName>${namespace}/base_link</bodyName>
+          <bodyName>base_link</bodyName>
           <topicName>imu</topicName>
           <serviceName>imu_service</serviceName>
@@ -242,5 +230,5 @@
       <plugin name="ground_truth_odometry" filename="libgazebo_ros_p3d.so">
         <robotNamespace>/${namespace}</robotNamespace>
-        <bodyName>${namespace}/base_link</bodyName>
+        <bodyName>base_link</bodyName>
         <topicName>ground_truth/odometry</topicName>
         <frameName>/world</frameName>

File: urdf/rotors/dji_m100.urdf.xacro (robot description, xacro)
@@ -1,4 +1,7 @@
 <?xml version="1.0"?>
 <robot name="dji_m100" xmlns:xacro="http://ros.org/wiki/xacro">
+  <xacro:arg name="robot_namespace" default=""/>
+  <xacro:arg name="complex_visualization_supported" default="true"/>
+  <xacro:property name="namespace" value="$(arg robot_namespace)" />
   <!-- Instantiate dji_m100 "mechanics" -->
   <xacro:include filename="$(find dji_m100_description)/urdf/dji_m100_base.xacro" />

Commit message: Fix collision, which was resulting in jittering.

File: urdf/dji_m100_base.xacro (robot description, xacro)
@@ -8,6 +8,4 @@
   <xacro:property name="rotor_velocity_slowdown_sim" value="10" />
   <xacro:property name="mass" value="2.355" /> <!-- [kg] -->
-  <xacro:property name="body_width" value="0.3" /> <!-- [m] / This value is not important since we've already provided the mesh. -->
-  <xacro:property name="body_height" value="0.16" /> <!-- [m] / This value is not important since we've already provided the mesh. -->
   <xacro:property name="mass_rotor" value="0.08" /> <!-- [kg] -->
   <xacro:property name="arm_length" value="0.17" /> <!-- [m] -->

File: urdf/rotors/dji_m100_multirotors.xacro (robot description, xacro)
@@ -19,4 +19,6 @@
 -->
 <robot xmlns:xacro="http://ros.org/wiki/xacro">
+   <xacro:property name="body_width" value="0.3" />
+  <xacro:property name="body_height" value="0.16" />
   <!-- Macro for the inertia of a box -->
   <xacro:macro name="box_inertia" params="x y z mass">
@@ -58,5 +60,5 @@
         <origin xyz="0 0 0" rpy="0 0 0" />
         <geometry>
-          <mesh filename="package://dji_m100_description/meshes/dji_m100/dji_m100_flipped_rotorless.stl"/>
+          <box size="${body_width} ${body_width} ${body_height}" /> <!-- [m] [m] [m] -->
         </geometry>
       </collision>
