Commit message: Add joint constraints on gimbal. Visualize tests in RViz.

File: urdf/gimbal.urdf.xacro (robot description, xacro)
@@ -28,8 +28,9 @@
             </collision>
         </link>
-        <joint name="gimbal_roll_joint" type="continuous">
+        <joint name="gimbal_roll_joint" type="revolute">
             <parent link="virtual_gimbal_link" />
             <child link="gimbal_roll_link" />
             <axis xyz="1 0 0" />
+            <limit effort="1000.0" lower="-0.48" upper="0.48" velocity="0.5" />
             <dynamics damping="0.0" friction="0.0" />
         </joint>
@@ -46,8 +47,9 @@
             </visual>
         </link>
-        <joint name="gimbal_pitch_joint" type="continuous">
+        <joint name="gimbal_pitch_joint" type="revolute">
             <parent link="gimbal_roll_link" />
             <child link="gimbal_pitch_link" />
             <axis xyz="0 1 0" />
+            <limit effort="1000.0" lower="-0.48" upper="0.48" velocity="0.5" />
             <dynamics damping="0.0" friction="0.0" />
         </joint>
@@ -68,4 +70,5 @@
             <child link="gimbal_yaw_link" />
             <axis xyz="0 0 1" />
+            <limit effort="1000.0" lower="-3.14" upper="3.14" velocity="0.5" />
             <dynamics damping="0.0" friction="0.0" />
         </joint>

Commit message: Improve structure of xacro files for gimbal.

File: urdf/gimbal.urdf.xacro (robot description, xacro)
@@ -1,4 +1,5 @@
 <?xml version="1.0"?>
 <robot xmlns:xacro="http://www.ros.org/wiki/xacro">
+    <xacro:include filename="$(find dji_m100_description)/urdf/gimbal_joints.xacro"/>
     <xacro:macro name="dji_m100_gimbal">
         <joint name="virtual_gimbal_joint" type="fixed">
@@ -28,11 +29,12 @@
             </collision>
         </link>
-        <joint name="gimbal_roll_joint" type="revolute">
-            <parent link="virtual_gimbal_link" />
-            <child link="gimbal_roll_link" />
-            <axis xyz="1 0 0" />
-            <limit effort="1000.0" lower="-0.48" upper="0.48" velocity="0.5" />
-            <dynamics damping="0.0" friction="0.0" />
-        </joint>
+        <revolute_gimbal_joint
+            name="gimbal_roll_joint"
+            parent="virtual_gimbal_link"
+            child="gimbal_roll_link"
+            lower_limit="-0.48"
+            upper_limit="0.48"
+            axis_xyz="1 0 0"
+            />
         <link name="gimbal_roll_link">
             <inertial>
@@ -47,11 +49,12 @@
             </visual>
         </link>
-        <joint name="gimbal_pitch_joint" type="revolute">
-            <parent link="gimbal_roll_link" />
-            <child link="gimbal_pitch_link" />
-            <axis xyz="0 1 0" />
-            <limit effort="1000.0" lower="-0.48" upper="0.48" velocity="0.5" />
-            <dynamics damping="0.0" friction="0.0" />
-        </joint>
+        <revolute_gimbal_joint
+            name="gimbal_pitch_joint"
+            parent="gimbal_roll_link"
+            child="gimbal_pitch_link"
+            lower_limit="-0.48"
+            upper_limit="0.48"
+            axis_xyz="0 1 0"
+            />
         <link name="gimbal_pitch_link">
             <inertial>
@@ -66,11 +69,12 @@
             </visual>
         </link>
-        <joint name="gimbal_yaw_joint" type="continuous">
-            <parent link="gimbal_pitch_link" />
-            <child link="gimbal_yaw_link" />
-            <axis xyz="0 0 1" />
-            <limit effort="1000.0" lower="-3.14" upper="3.14" velocity="0.5" />
-            <dynamics damping="0.0" friction="0.0" />
-        </joint>
+        <revolute_gimbal_joint
+            name="gimbal_yaw_joint"
+            parent="gimbal_pitch_link"
+            child="gimbal_yaw_link"
+            lower_limit="-3.14"
+            upper_limit="3.14"
+            axis_xyz="0 0 1"
+            />
         <link name="gimbal_yaw_link">
             <inertial>

Commit message: Remove unnecessary virtual joint.

File: urdf/gimbal.urdf.xacro (robot description, xacro)
@@ -3,47 +3,32 @@
     <xacro:include filename="$(find dji_m100_description)/urdf/gimbal_joints.xacro"/>
     <xacro:macro name="dji_m100_gimbal">
-        <joint name="virtual_gimbal_joint" type="fixed">
-            <origin xyz="-0.1 0 -0.04" rpy="0 0 0"/>
-            <parent link="base_link"/>
-            <child link="virtual_gimbal_link"/>
-        </joint>
-        <gazebo reference="virtual_gimbal_joint">
-            <preserveFixedJoint>true</preserveFixedJoint>
-        </gazebo>
-        <link name="virtual_gimbal_link">
-            <inertial>
-                <mass value="0.0001" />
-                <origin xyz="0 0 0" rpy="0 0 0" />
-                <inertia ixx="0.0001" ixy="0" ixz="0" iyy="0.0001" iyz="0" izz="0.0001" />
-            </inertial>
-            <visual>
-                <geometry>
-                <box size="0.0001 0.0001 0.0001" />
-                </geometry>
-            </visual>
-            <collision>
-                <origin xyz="0 0 0" rpy="0 0 0" />
-                <geometry>
-                <mesh filename="package://dji_m100_description/meshes/dji_m100/gimbal.stl"/>
-                </geometry>
-            </collision>
-        </link>
         <revolute_gimbal_joint
             name="gimbal_roll_joint"
-            parent="virtual_gimbal_link"
+            parent="base_link"
             child="gimbal_roll_link"
             lower_limit="-0.48"
             upper_limit="0.48"
             axis_xyz="1 0 0"
+            origin_xyz="-0.1 0 -0.04"
             />
+        <transmission name="trans_roll">
+            <type>transmission_interface/SimpleTransmission</type>
+            <joint name="gimbal_roll_joint">
+                <hardwareInterface>hardware_interface/EffortJointInterface</hardwareInterface>
+            </joint>
+            <actuator name="motor_roll">
+                <hardwareInterface>hardware_interface/EffortJointInterface</hardwareInterface>
+                <mechanicalReduction>1</mechanicalReduction>
+            </actuator>
+        </transmission>
         <link name="gimbal_roll_link">
             <inertial>
-                <mass value="0.0001" />
-                <origin xyz="0 0 0" rpy="0 0 0" />
-                <inertia ixx="0.0001" ixy="0" ixz="0" iyy="0.0001" iyz="0" izz="0.0001" />
+                <mass value="0.1" />
+                <origin xyz="-0.1 0 -0.04" rpy="0 0 0" />
+                <inertia ixx="0.0" ixy="0" ixz="0" iyy="0.0" iyz="0" izz="0.0" />
             </inertial>
             <visual>
                 <geometry>
-                <box size="0.0001 0.0001 0.0001" />
+                    <box size="0.0001 0.0001 0.0001" />
                 </geometry>
             </visual>
@@ -56,10 +41,21 @@
             upper_limit="0.48"
             axis_xyz="0 1 0"
+            origin_xyz="0 0 0"
             />
+        <transmission name="trans_pitch">
+            <type>transmission_interface/SimpleTransmission</type>
+            <joint name="gimbal_pitch_joint">
+                <hardwareInterface>hardware_interface/EffortJointInterface</hardwareInterface>
+            </joint>
+            <actuator name="motor_pitch">
+                <hardwareInterface>hardware_interface/EffortJointInterface</hardwareInterface>
+                <mechanicalReduction>1</mechanicalReduction>
+            </actuator>
+        </transmission>
         <link name="gimbal_pitch_link">
             <inertial>
-                <mass value="0.0001" />
+                <mass value="0.1" />
                 <origin xyz="0 0 0" rpy="0 0 0" />
-                <inertia ixx="0.0001" ixy="0" ixz="0" iyy="0.0001" iyz="0" izz="0.0001" />
+                <inertia ixx="0.0" ixy="0" ixz="0" iyy="0.0" iyz="0" izz="0.0" />
             </inertial>
             <visual>
@@ -76,15 +72,26 @@
             upper_limit="3.14"
             axis_xyz="0 0 1"
+            origin_xyz="0 0 0"
             />
+        <transmission name="trans_yaw">
+            <type>transmission_interface/SimpleTransmission</type>
+            <joint name="gimbal_yaw_joint">
+                <hardwareInterface>hardware_interface/EffortJointInterface</hardwareInterface>
+            </joint>
+            <actuator name="motor_yaw">
+                <hardwareInterface>hardware_interface/EffortJointInterface</hardwareInterface>
+                <mechanicalReduction>1</mechanicalReduction>
+            </actuator>
+        </transmission>
         <link name="gimbal_yaw_link">
             <inertial>
-                <mass value="0.0001" />
+                <mass value="0.1" />
                 <origin xyz="0 0 0" rpy="0 0 ${-M_PI}" />
-                <inertia ixx="0.0001" ixy="0" ixz="0" iyy="0.0001" iyz="0" izz="0.0001" />
+                <inertia ixx="0.0" ixy="0" ixz="0" iyy="0.0" iyz="0" izz="0.0" />
             </inertial>
             <visual>
                 <origin xyz="0 0 0" rpy="0 0 ${-M_PI}" />
                 <geometry>
-                <mesh filename="package://dji_m100_description/meshes/dji_m100/gimbal.dae"/>
+                    <mesh filename="package://dji_m100_description/meshes/dji_m100/gimbal.dae"/>
                 </geometry>
             </visual>

File: urdf/gimbal_joints.xacro (robot description, xacro)
@@ -1,11 +1,12 @@
 <?xml version="1.0" ?>
 <robot xmlns:xacro="http://www.ros.org/wiki/xacro">
-    <xacro:macro name="revolute_gimbal_joint" params="name axis_xyz parent child upper_limit lower_limit">
+    <xacro:macro name="revolute_gimbal_joint" params="name axis_xyz parent child upper_limit lower_limit origin_xyz">
         <joint name="${name}" type="revolute">
             <parent link="${parent}" />
             <child link="${child}" />
             <axis xyz="${axis_xyz}" />
-            <limit effort="1000.0" lower="${lower_limit}" upper="${upper_limit}" velocity="0.5" />
+            <limit effort="1000.0" lower="${lower_limit}" upper="${upper_limit}" velocity="1.5" />
             <dynamics damping="0.0" friction="0.0" />
+            <origin xyz="${origin_xyz}" rpy="0 0 0"/>
         </joint>
     </xacro:macro>

Commit message: Add transmission to custom gimbal joint.

File: urdf/gimbal.urdf.xacro (robot description, xacro)
@@ -12,14 +12,4 @@
             origin_xyz="-0.1 0 -0.04"
             />
-        <transmission name="trans_roll">
-            <type>transmission_interface/SimpleTransmission</type>
-            <joint name="gimbal_roll_joint">
-                <hardwareInterface>hardware_interface/EffortJointInterface</hardwareInterface>
-            </joint>
-            <actuator name="motor_roll">
-                <hardwareInterface>hardware_interface/EffortJointInterface</hardwareInterface>
-                <mechanicalReduction>1</mechanicalReduction>
-            </actuator>
-        </transmission>
         <link name="gimbal_roll_link">
             <inertial>
@@ -43,14 +33,4 @@
             origin_xyz="0 0 0"
             />
-        <transmission name="trans_pitch">
-            <type>transmission_interface/SimpleTransmission</type>
-            <joint name="gimbal_pitch_joint">
-                <hardwareInterface>hardware_interface/EffortJointInterface</hardwareInterface>
-            </joint>
-            <actuator name="motor_pitch">
-                <hardwareInterface>hardware_interface/EffortJointInterface</hardwareInterface>
-                <mechanicalReduction>1</mechanicalReduction>
-            </actuator>
-        </transmission>
         <link name="gimbal_pitch_link">
             <inertial>
@@ -74,14 +54,4 @@
             origin_xyz="0 0 0"
             />
-        <transmission name="trans_yaw">
-            <type>transmission_interface/SimpleTransmission</type>
-            <joint name="gimbal_yaw_joint">
-                <hardwareInterface>hardware_interface/EffortJointInterface</hardwareInterface>
-            </joint>
-            <actuator name="motor_yaw">
-                <hardwareInterface>hardware_interface/EffortJointInterface</hardwareInterface>
-                <mechanicalReduction>1</mechanicalReduction>
-            </actuator>
-        </transmission>
         <link name="gimbal_yaw_link">
             <inertial>

File: urdf/gimbal_joints.xacro (robot description, xacro)
@@ -6,8 +6,18 @@
             <child link="${child}" />
             <axis xyz="${axis_xyz}" />
-            <limit effort="1000.0" lower="${lower_limit}" upper="${upper_limit}" velocity="1.5" />
+            <limit effort="1000.0" lower="${lower_limit}" upper="${upper_limit}" velocity="2.5" />
             <dynamics damping="0.0" friction="0.0" />
             <origin xyz="${origin_xyz}" rpy="0 0 0"/>
         </joint>
+        <transmission name="trans_${name}">
+            <type>transmission_interface/SimpleTransmission</type>
+            <joint name="${name}">
+                <hardwareInterface>hardware_interface/EffortJointInterface</hardwareInterface>
+            </joint>
+            <actuator name="${name}">
+                <hardwareInterface>hardware_interface/EffortJointInterface</hardwareInterface>
+                <mechanicalReduction>1</mechanicalReduction>
+            </actuator>
+        </transmission>
     </xacro:macro>
 </robot>

Commit message: Gimball mass and inertia made so that the robot base is not disturbed catasthropically.

File: urdf/gimbal.urdf.xacro (robot description, xacro)
@@ -3,19 +3,48 @@
     <xacro:include filename="$(find dji_m100_description)/urdf/gimbal_joints.xacro"/>
     <xacro:property name="M_PI" value="3.14"/>
+    <material name="black">
+        <color rgba="0 0 0 1"/>
+    </material>
     <xacro:macro name="dji_m100_gimbal">
-        <revolute_gimbal_joint
+        <joint name="gimbal_base_joint" type="fixed">
+            <parent link="base_link"/>
+            <child link="gimbal_base_plate" />
+        </joint>
+        <gazebo reference="gimbal_base_joint">
+            <preserveFixedJoint>true</preserveFixedJoint>
+        </gazebo>
+        <link name="gimbal_base_plate">
+            <visual>
+                <geometry>
+                    <box size="0.01 0.01 0.06"/>
+                </geometry>
+                <origin xyz="0.0 0 -0.03" rpy="0 ${-75 * M_PI/180.0} 0"/>
+                <material name="black"/>
+            </visual>
+            <collision>
+                <geometry>
+                    <box size="0.01 0.01 0.06"/>
+                </geometry>
+                <origin xyz="0.0 0 -0.03" rpy="0 ${-75 * M_PI/180.0} 0"/>
+            </collision>
+            <inertial>
+                <mass value="0.01"/>
+                <inertia ixx="0.0000125" ixy="0.0" ixz="0.0" iyy="0.0000125" iyz="0.0" izz="0.0000125"/>
+            </inertial>
+        </link>
+         <revolute_gimbal_joint
             name="gimbal_roll_joint"
-            parent="base_link"
+            parent="gimbal_base_plate"
             child="gimbal_roll_link"
             lower_limit="-0.48"
             upper_limit="0.48"
             axis_xyz="1 0 0"
-            origin_xyz="-0.1 0 -0.04"
+            origin_xyz="0.05 0 -0.04"
             />
         <link name="gimbal_roll_link">
             <inertial>
-                <mass value="0.1" />
-                <origin xyz="-0.1 0 -0.04" rpy="0 0 0" />
-                <inertia ixx="0.0" ixy="0" ixz="0" iyy="0.0" iyz="0" izz="0.0" />
+                <origin xyz="0 0 0" rpy="0 0 0" />
+                <mass value="0.01"/>
+                <inertia ixx="0.0000125" ixy="0.0" ixz="0.0" iyy="0.0000125" iyz="0.0" izz="0.0000125"/>
             </inertial>
             <visual>
@@ -36,7 +65,7 @@
         <link name="gimbal_pitch_link">
             <inertial>
-                <mass value="0.1" />
                 <origin xyz="0 0 0" rpy="0 0 0" />
-                <inertia ixx="0.0" ixy="0" ixz="0" iyy="0.0" iyz="0" izz="0.0" />
+                <mass value="0.01"/>
+                <inertia ixx="0.0000125" ixy="0.0" ixz="0.0" iyy="0.0000125" iyz="0.0" izz="0.0000125"/>
             </inertial>
             <visual>
@@ -50,6 +79,6 @@
             parent="gimbal_pitch_link"
             child="gimbal_yaw_link"
-            lower_limit="-3.14"
-            upper_limit="3.14"
+            lower_limit="-1.57"
+            upper_limit="1.57"
             axis_xyz="0 0 1"
             origin_xyz="0 0 0"
@@ -57,46 +86,27 @@
         <link name="gimbal_yaw_link">
             <inertial>
-                <mass value="0.1" />
-                <origin xyz="0 0 0" rpy="0 0 ${-M_PI}" />
-                <inertia ixx="0.0" ixy="0" ixz="0" iyy="0.0" iyz="0" izz="0.0" />
+                <origin xyz="0 0 0" rpy="0 0 0" />
+                <mass value="0.01"/>
+                <inertia ixx="0.0000125" ixy="0.0" ixz="0.0" iyy="0.0000125" iyz="0.0" izz="0.0000125"/>
             </inertial>
             <visual>
-                <origin xyz="0 0 0" rpy="0 0 ${-M_PI}" />
+                <origin xyz="0 0 0" rpy="0 0 0" />
                 <geometry>
                     <mesh filename="package://dji_m100_description/meshes/dji_m100/gimbal.dae"/>
                 </geometry>
             </visual>
-            <collision>
-                <origin xyz="0 0 0" rpy="0 0 ${-M_PI}" />
-                <geometry>
-                <mesh filename="package://dji_m100_description/meshes/dji_m100/gimbal.stl"/>
-                </geometry>
-            </collision>
         </link>
-        <joint name="camera_joint" type="continuous">
-            <parent link="gimbal_yaw_link" />
-            <child link="camera_link" />
-            <axis xyz="0 0 1" />
-            <dynamics damping="0.0" friction="0.0" />
-        </joint>
-        <link name="camera_link">
-        </link>
-        <joint name="camera_optical_joint" type="fixed">
-            <origin xyz="0 0 0" rpy="${-M_PI/2} 0.0 ${-M_PI/2}" />
-            <parent link="camera_link" />
-            <child link="camera_optical_frame"/>
-        </joint>
-        <gazebo reference="camera_optical_joint">
-            <preserveFixedJoint>true</preserveFixedJoint>
+        <gazebo>
+            <plugin name="gazebo_ros_control" filename="libgazebo_ros_control.so">
+            </plugin>
         </gazebo>
-        <link name="camera_optical_frame">
-        </link>
+        <gazebo reference="gimbal_base_plate">
+            <material>Gazebo/FlatBlack</material>
+        </gazebo>
         <gazebo reference="gimbal_yaw_link">
             <sensor type="camera" name="camera_camera_sensor">
                 <update_rate>10</update_rate>
                 <camera>
-                <!-- <pose>0.027 0 -0.027 0 1.57 0</pose> -->
-                <!-- <pose>0.027 0 -0.027 0 1.57 0</pose> -->
-                <pose>0.107 0 -0.227 0 0 ${M_PI}</pose>
+                <pose>0.107 0 -0.227 0 0 0</pose>
                 <horizontal_fov>${94 * M_PI/180.0}</horizontal_fov>
                 <image>

File: urdf/gimbal_joints.xacro (robot description, xacro)
@@ -6,5 +6,5 @@
             <child link="${child}" />
             <axis xyz="${axis_xyz}" />
-            <limit effort="1000.0" lower="${lower_limit}" upper="${upper_limit}" velocity="2.5" />
+            <limit effort="0.005" lower="${lower_limit}" upper="${upper_limit}" velocity="0.2" />
             <dynamics damping="0.0" friction="0.0" />
             <origin xyz="${origin_xyz}" rpy="0 0 0"/>
